File: Hardware/DRV8304_FOC.kicad_pcb (KiCad board)
At the start: 4 copper layers, 55 x 55 mm, 70 parts, among them J1 Conn_01x01_Pin, J2 Conn_01x01_Pin, J3 Conn_01x01_Pin, J5 Conn_02x07_Odd_Even, Q1 SIRA18ADP, Q2 SIRA18ADP, Q3 SIRA18ADP, Q4 SIRA18ADP, Q5 SIRA18ADP, Q6 SIRA18ADP, SW2 SW_Push, U1 TPS565208, U3 DRV8304HRHAR, U4 STM32F412CEUx, U6 AS5047P, Y1 Crystal_GND23

Commit message: Regular Commit
Parts:
- removed C27: 100uF, Capacitor_SMD:CP_Elec_6.3x7.7
- removed J5: Conn_02x07_Odd_Even, Connector_PinHeader_1.27mm:PinHeader_2x07_P1.27mm_Vertical_SMD
- added C1: C, Capacitor_SMD:C_1206_3216Metric, F.Cu at (170.9, 119.8)
- added C2: C, Capacitor_SMD:C_1206_3216Metric, F.Cu at (169.2, 118.1)
- added C9: C, Capacitor_SMD:C_1206_3216Metric, F.Cu at (167.3, 116.1)
- added J6: Conn_01x01_Pin, Connector_Wire:SolderWirePad_1x01_SMD_1x2mm, F.Cu at (123.1, 90.9)
- added J7: Conn_01x01_Pin, Connector_Wire:SolderWirePad_1x01_SMD_1x2mm, F.Cu at (123.1, 88.3)
- added J8: Conn_01x01_Pin, Connector_Wire:SolderWirePad_1x01_SMD_1x2mm, F.Cu at (123.1, 85.8)
- added J9: TC2070, Connector:Tag-Connect_TC2070-IDC-FP_2x07_P1.27mm_Vertical, F.Cu at (131.6, 101.8)
- H1, H2, H3, H4: footprint MountingHole:MountingHole_3.2mm_M3_DIN965_Pad -> MountingHole:MountingHole_3.2mm_M3_ISO14580_Pad_TopOnly; moved to B.Cu
- moved H3 67.9 mm to (145.1, 104.2), turned to 180 degrees
- moved H2 58.6 mm to (160.7, 104.4), turned to 180 degrees
- moved H4 53.2 mm to (153.1, 94.7), turned to 180 degrees
- moved C22 49.3 mm to (158.6, 124.5), turned to -90 degrees
- moved R18 47.2 mm to (148.0, 123.2), turned to 0 degrees
- moved R16 45.8 mm to (146.1, 121.9), turned to 0 degrees
- moved R17 45.7 mm to (148.0, 121.9), turned to 0 degrees
- moved J2 43.7 mm to (129.2, 115.3), turned to -60 degrees
- moved C20 42.1 mm to (150.9, 127.7)
- moved C21 41.4 mm to (157.0, 126.8), turned to 180 degrees
- moved J3 41.1 mm to (130.0, 116.6), turned to -60 degrees
- moved R20 40.2 mm to (148.0, 125.8), turned to 0 degrees
- moved R19 37.6 mm to (146.1, 123.2), turned to 0 degrees
- moved R25 37.6 mm to (149.5, 127.5), turned to -90 degrees
- moved R21 37.0 mm to (146.1, 125.8), turned to 0 degrees
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Connections:
- C3 pad 1: VIN -> Vin
- C4 pad 1: VIN -> Vin
- C5 pad 1: VIN -> Vin
- C7 pad 1: 1V8 -> 3V3
- C8 pad 1: 1V8 -> 3V3
- L1 pad 2: 1V8 -> 3V3
- Q2 pad 1: Net-(Q2-S-Pad1) -> SPA
- Q2 pad 2: Net-(Q2-S-Pad1) -> SPA
- Q2 pad 3: Net-(Q2-S-Pad1) -> SPA
- Q4 pad 1: Net-(Q4-S-Pad1) -> SPB
- Q4 pad 2: Net-(Q4-S-Pad1) -> SPB
- Q4 pad 3: Net-(Q4-S-Pad1) -> SPB
- Q6 pad 1: Net-(Q6-S-Pad1) -> SPC
- Q6 pad 2: Net-(Q6-S-Pad1) -> SPC
- Q6 pad 3: Net-(Q6-S-Pad1) -> SPC
- R1 pad 2: VIN -> Vin
- R11 pad 1: Net-(Q2-S-Pad1) -> SPA
- R12 pad 1: Net-(Q4-S-Pad1) -> SPB
- R13 pad 1: Net-(Q6-S-Pad1) -> SPC
- R3 pad 1: 1V8 -> 3V3
- TP1 pad 1: INHA -> INHC
- TP5 pad 1: INHC -> INHA
- TP7 pad 1: ISENSE_C -> ISENSE_A
- TP9 pad 1: ISENSE_A -> ISENSE_C
- U1 pad 3: VIN -> Vin
- U3 pad 10: SNA -> GND
- U3 pad 11: SNB -> GND
- U3 pad 20: SNC -> GND
- U3 pad 21: ISENSE_C -> ISENSE_A
- U3 pad 23: ISENSE_A -> ISENSE_C
- U3 pad 34: INHA -> INHC
- U3 pad 38: INHC -> INHA
- Y1 pad 2: Net-(Y1-G-Pad2) -> GND
- Y1 pad 3: Net-(Y1-G-Pad2) -> GND
Routing:
- net SHC: track 0.00 -> 49.4 mm, vias 0 -> 17
- net SHB: track 0.00 -> 49.2 mm, vias 0 -> 17
- net GHB: track 0.00 -> 47.4 mm, vias 1 -> 2
- net SPI_MISO: track 0.00 -> 46.7 mm, vias 0 -> 2
- net GHC: track 0.00 -> 46.4 mm, vias 0 -> 2
- net GLC: track 0.00 -> 40.6 mm, vias 0 -> 2
- net GLB: track 0.00 -> 40.0 mm, vias 0 -> 2
- net GHA: track 0.00 -> 38.7 mm, vias 0 -> 2
- net SHA: track 0.00 -> 38.0 mm, vias 0 -> 17
- net SPI_MOSI: track 0.00 -> 37.6 mm
- net SPC: track 0.00 -> 37.2 mm, vias 0 -> 2
- net INHA: track 6.40 -> 42.2 mm, vias 0 -> 2
- net SPB: track 0.00 -> 33.8 mm, vias 0 -> 2
- net SPI_SCK: track 0.00 -> 32.7 mm, vias 0 -> 2
- net INHB: track 6.03 -> 38.1 mm, vias 0 -> 2
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- added copper zone on F.Cu, net 3V3
- added copper zone on F.Cu, net SHA
- added copper zone on F.Cu, net SHB
- added copper zone on F.Cu, net SHC
- added copper zone on F.Cu, net Vin
- added copper zone on In2.Cu, net Vin
- removed copper zone on F.Cu, net 1V8
- removed copper zone on F.Cu, net VIN
Other:
- board size 55 x 55 mm -> 61 x 61 mm

Commit message: Regular Commit
Parts:
- moved C23 3.89 mm to (135.1, 120.1)
- moved C24 3.82 mm to (132.2, 117.3)
- moved R12 1.23 mm to (166.1, 94.0)
- moved R11 1.10 mm to (169.2, 106.6)
- moved C30 0.28 mm to (152.2, 99.6), turned to 180 degrees
Routing:
- net GND: track 8.98 -> 36.0 mm, vias 12 -> 38
- net 3V3: track 24.7 -> 41.6 mm, vias 2 -> 18
- net SPI_~{SS}: track 0.00 -> 14.3 mm, vias 0 -> 2
- net SPI_MISO: track 46.7 -> 36.5 mm
- net SPI_MOSI: track 37.6 -> 32.2 mm
- net SPI_SCK: track 32.7 -> 28.2 mm
- net SHC: track 49.4 -> 53.6 mm
- net SPB: track 33.8 -> 37.1 mm
- net Net-(U4-VCAP_1): track 0.00 -> 3.09 mm
- net SPC: track 37.2 -> 39.4 mm
- net Net-(U4-PH1): track 5.71 -> 7.33 mm
- net Net-(U4-PH0): track 5.72 -> 7.30 mm
- net SPA: track 24.3 -> 25.8 mm
- net GHB: track 47.4 -> 48.4 mm
- net GHC: track 46.4 -> 47.1 mm
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- added copper zone on In2.Cu, net 3V3
- added copper zone on F.Cu, net SPA
- added copper zone on F.Cu, net SPB
- added copper zone on F.Cu, net SPC

Commit message: Commit for review
Parts:
- removed J6, J7, J8: Conn_01x01_Pin, Connector_Wire:SolderWirePad_1x01_SMD_1x2mm
- moved TP1 0.40 mm to (152.5, 127.6)
- moved TP3 0.40 mm to (153.9, 127.6)
- moved TP5 0.40 mm to (155.3, 127.6)
Connections:
- U3 pad V: (no net) -> GND
Routing:
- net GND: track 36.0 -> 49.7 mm, vias 38 -> 127
- net 3V3: track 41.6 -> 49.7 mm, vias 18 -> 23
- net /~{RST}: track 27.3 -> 34.0 mm, vias 2 -> 3
- net Net-(U3-CAL): track 0.00 -> 3.01 mm
- net GHC: track 47.1 -> 50.0 mm
- net GLB: track 40.0 -> 42.6 mm
- net Net-(U3-DVDD): track 0.00 -> 2.59 mm
- net GLA: track 27.8 -> 30.0 mm
- net GLC: track 40.6 -> 42.5 mm
- net GHB: track 48.4 -> 50.2 mm
- net SHA: track 38.0 -> 36.2 mm
- net INHC: track 33.9 -> 33.3 mm
- net SPI_~{SS}: track 14.3 -> 13.8 mm
- net Vin: vias 40 -> 49
Other:
- board size 61 x 61 mm -> 60.9 x 60.9 mm

Commit message: FAB OUT GERBER
Parts:
- Y1: value Crystal_GND23 -> Crystal_GND24
- moved Y1 1.61 mm to (133.0, 120.0), turned to -45 degrees
- moved C24 0.70 mm to (132.9, 117.3), turned to -45 degrees
- moved C23 0.50 mm to (135.5, 119.8), turned to 135 degrees
- moved R2 0.13 mm to (134.8, 88.4)
- moved R1 0.11 mm to (134.8, 90.4)
- moved R3 0.11 mm to (134.8, 89.4)
- moved J2 0.10 mm to (129.2, 115.2)
Connections:
- Y1 pad 3: GND -> Net-(U4-PH1)
- Y1 pad 4: Net-(U4-PH1) -> GND
Routing:
- net GND: track 49.7 -> 44.7 mm
- net Net-(U4-PH0): track 7.30 -> 9.17 mm
- net Net-(U4-PH1): track 7.33 -> 8.51 mm
- added copper zone on B.Cu, net SHA
- added copper zone on B.Cu, net SHB
- added copper zone on B.Cu, net SHC
- added copper zone on B.Cu, net Vin
Other:
- board text added: "G"
- board text added: "RX"
- board text added: "TX"
