File: motherboard/motherboard.kicad_pcb (KiCad board)
At the start: 4 copper layers, 50 x 50 mm, 50 parts, among them IC1 TCAN3403DRQ1, J1 Conn_01x01_Pin, J1 Conn_02x07_Odd_Even, J10 Conn_01x01_Pin, J11 Conn_01x01_Pin, J12 Conn_01x01_Pin, J2 Conn_01x01_Pin, J3 Conn_01x01_Pin, J4 Conn_01x01_Pin, J5 Conn_01x01_Pin, J6 Conn_01x01_Pin, J7 Conn_01x01_Pin, J8 Conn_01x01_Pin, J9 Conn_01x01_Pin, SW1 SW_Push, U1 TPS565208, U2 STM32F723VCTx, Y1 Crystal_GND24

Commit message: update
Parts:
- moved J1 24.7 mm to (214.0, 61.0)
- moved Y1 6.98 mm to (206.7, 90.0), turned to -90 degrees
- moved C1 5.18 mm to (203.8, 67.9)
- moved C13 5.18 mm to (198.2, 60.7)
- moved C3 5.18 mm to (203.8, 66.4)
- moved L1 5.18 mm to (198.2, 64.2)
- moved R1 5.18 mm to (206.7, 64.2)
- moved R3 5.18 mm to (206.7, 65.2)
- moved U1 5.18 mm to (203.8, 64.2)
- moved C12 5.18 mm to (198.2, 58.7)
- moved C7 5.18 mm to (204.8, 62.0)
- moved C2 5.18 mm to (203.8, 69.9)
- moved R2 5.18 mm to (206.7, 66.1)
- moved IC1 3.92 mm to (233.1, 63.9)
- moved J5 2.59 mm to (236.4, 90.0)
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Connections:
- net CANH renamed CAN_P
- net CANL renamed CAN_N
- J1 pad 13: unconnected-(J1-Pin_13-Pad13) -> /VCP_RX
- J1 pad 14: unconnected-(J1-Pin_14-Pad14) -> /VCP_TX
- U2 pad 97: unconnected-(U2-PE0-Pad97) -> /VCP_RX
- U2 pad 98: unconnected-(U2-PE1-Pad98) -> /VCP_TX
Routing:
- net CAN_P: track 0.00 -> 3.03 mm
- net CAN_N: track 0.00 -> 3.03 mm
