File: motherboard/motherboard.kicad_sch (KiCad schematic)
At the start: 48 parts, among them IC1 TCAN3403DRQ1, J1 Conn_02x07_Odd_Even, J10 Conn_01x01_Pin, J11 Conn_01x01_Pin, J12 Conn_01x01_Pin, J2 Conn_01x01_Pin, J3 Conn_01x01_Pin, J4 Conn_01x01_Pin, J5 Conn_01x01_Pin, J6 Conn_01x01_Pin, J7 Conn_01x01_Pin, J8 Conn_01x01_Pin, J9 Conn_01x01_Pin, SW1 SW_Push, U1 TPS565208, U2 STM32F723VCTx, Y1 Crystal_GND24

Commit message: update
Connections:
- net VCP_RX: now reaches J1.13 (Pin_13)
- net VCP_RX: now also U2.97 (PE0)
- net VCP_TX: now reaches J1.14 (Pin_14)
- net VCP_TX: now also U2.98 (PE1)
- net CANH renamed CAN_P
- net CANL renamed CAN_N
- no-connect marks 76 -> 72
Other:
- moved on the sheet: IC1
